File: avionics.sch (KiCad schematic (older format))
At the start: 11 parts, among them P1 Ant, P2 GPS Connector, P7 D24V5F3, U2 RFM22, U3 WeMos_mini, U4 Teensy_3.1

Commit message: Initial design with traces - a little bit gross
Connections:
- net Cont1 renamed Firing_circuits/Cont1
Changed lines of the file:
@@
 	11100 1900 11100 2050
 Wire Wire Line
-	11100 2350 11100 2500
-Wire Wire Line
 	11100 2800 11100 2900
-Wire Wire Line
-	10550 2600 10900 2600
-Wire Wire Line
-	10900 2600 10900 2450
-Wire Wire Line
-	10900 2450 11100 2450
-Connection ~ 11100 2450
 $Comp
 L GND #PWR08
@@
 Wire Wire Line
 	8850 5150 9100 5150
-Text Label 8850 5250 2    60   ~ 0
-Cont1
 Text Label 10550 5200 0    60   ~ 0
 Fire1
@@
 Aux2
 Wire Wire Line
-	9100 5250 8850 5250
+	8450 5250 9100 5250
 Wire Wire Line
 	10450 5700 10550 5700
@@
 Wire Wire Line
 	10800 3200 10800 3350
-Text Label 8500 3050 2    60   ~ 0
-Cont1
 Wire Wire Line
 	8550 1850 8500 1850
 Wire Wire Line
-	8500 3050 8550 3050
+	8450 3050 8550 3050
 Wire Wire Line
 	10550 3200 10800 3200
@@
 	2150 3600 2400 3600
 Connection ~ 2850 3600
+Wire Wire Line
+	11100 2350 11100 2500
+Wire Wire Line
+	11100 2450 10950 2450
+Wire Wire Line
+	10950 2450 10950 2600
+Wire Wire Line
+	10950 2600 10550 2600
+Connection ~ 11100 2450
+Wire Wire Line
+	8450 3050 8450 5250
 $EndSCHEMATC
